File: VCO/VCO_selfetch/power.kicad_sch (KiCad schematic)
At the start: 17 parts, among them U1 40106, U2 TL074, U3 TL074, U4 TL074, U5 TL074, U6 TL074, U7 TL074, U8 TL074

Commit message: footprint WIP
Parts:
- C25: renamed from C17; footprint (none) -> Capacitor_SMD:C_0402_1005Metric_Pad0.74x0.62mm_HandSolder
- C26, C27, C28, C29, C30, C31, C32, C33: renamed from C17; footprint (none) -> Capacitor_SMD:C_0603_1608Metric_Pad1.08x0.95mm_HandSolder
- U1, U2, U3, U4, U5, U6, U7, U8: footprint (none) -> Package_DIP:DIP-14_W7.62mm_Socket
