File: VCO/VCO_selfetch/simple_VCOs.kicad_sch (KiCad schematic)
At the start: 96 parts

Commit message: continue
Parts:
- gave numbers to parts that had none: 88

Commit message: footprint WIP
Parts:
- removed Q19, Q20, Q21: BC558, Package_TO_SOT_THT:TO-92_Inline, symbol Transistor_BJT:BC558
- removed Q22, Q23, Q24: BC548, Package_TO_SOT_THT:TO-92_Inline, symbol Transistor_BJT:BC548
- added Q19, Q21, Q23: BC858, Package_TO_SOT_SMD:SOT-23, symbol Transistor_BJT:BC858
- added Q20, Q22, Q24: BC848, Package_TO_SOT_SMD:SOT-23, symbol Transistor_BJT:BC848
- C16, C17, C18, C19, C20, C21, C22, C23, C24: footprint (none) -> Capacitor_SMD:C_0402_1005Metric_Pad0.74x0.62mm_HandSolder
- D16, D17, D18: footprint Diode_THT:D_DO-35_SOD27_P7.62mm_Horizontal -> Diode_SMD:D_SOD-123
- R100, R101, R102, R103, R104, R105, R106, R107, R108, R109, R111, R113, R115, R116, R117, R118, R119, R120, R121, R122, R123, R124, R125, R126, R127, R128, R129, R130, R131, R132, R133, R134, R135, R136, R137, R138, R139, R140, R141, R142, R143, R144, TH13, TH14, TH15, TH16, TH17, TH18, TH19, TH20, TH21: footprint (none) -> Resistor_SMD:R_0603_1608Metric_Pad0.98x0.95mm_HandSolder
- R110, R112, R114: footprint (none) -> Potentiometer_THT:Potentiometer_Bourns_3296W_Vertical
- RV16, RV17, RV18, RV19, RV20, RV21, RV22, RV23, RV24, RV25, RV26, RV27: footprint (none) -> Connector_PinHeader_2.54mm:PinHeader_1x03_P2.54mm_Vertical
- U1, U6, U7, U8: footprint (none) -> Package_DIP:DIP-14_W7.62mm_Socket
Connections:
- net -12V: now also Q19.3 (C), Q21.3 (C), Q23.3 (C)
- net GND: now also Q20.2 (E), Q22.2 (E), Q24.2 (E)
- net at R109.1, TH13.2, TH16.2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: now also Q19.1 (B)
- net at R115.2: now also Q19.2 (E), Q20.1 (B)
- net at C17.2, D17.1 (K), U1.11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: now also Q22.3 (C)
- net at C18.2, D18.1 (K), U1.13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: now also Q24.3 (C)
- net at R116.2: now also Q21.2 (E), Q22.1 (B)
- net at R117.2: now also Q23.2 (E), Q24.1 (B)
- net at R111.1, TH14.2, TH17.2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: now also Q21.1 (B)
- net at C16.2, D16.1 (K), U1.9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: now also Q20.3 (C)
- net at R113.1, TH15.2, TH18.2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: now also Q23.1 (B)

Commit message: all save
Parts:
- added J17: CV_in_4, Connector_PinHeader_2.54mm:PinHeader_1x02_P2.54mm_Vertical, symbol Connector:Conn_01x02_Pin
- added J18: CV_in_5, Connector_PinHeader_2.54mm:PinHeader_1x02_P2.54mm_Vertical, symbol Connector:Conn_01x02_Pin
- added J19, J22: CV_in_6, Connector_PinHeader_2.54mm:PinHeader_1x02_P2.54mm_Vertical, symbol Connector:Conn_01x02_Pin
- added J20: PWMMOD_in_4, Connector_PinHeader_2.54mm:PinHeader_1x02_P2.54mm_Vertical, symbol Connector:Conn_01x02_Pin
- added J21: PWMMOD_in_5, Connector_PinHeader_2.54mm:PinHeader_1x02_P2.54mm_Vertical, symbol Connector:Conn_01x02_Pin
Connections:
- net CV_IN4: now also J17.1 (Pin_1)
- net CV_IN5: now also J18.1 (Pin_1)
- net CV_IN6: now also J19.1 (Pin_1)
- net GND: now also J17.2 (Pin_2), J18.2 (Pin_2), J19.2 (Pin_2), J20.2 (Pin_2), J21.2 (Pin_2), J22.2 (Pin_2)
- net PWM_MOD4: now also J20.1 (Pin_1)
- net PWM_MOD5: now also J21.1 (Pin_1)
- net PWM_MOD6: now also J22.1 (Pin_1)
