File: VCO/VCO_single_osc/VCO_selfetch.kicad_pcb (KiCad board)
At the start: 4 copper layers, 62 parts, among them J11 CV_in_1, J14 PWMMOD_in_1, J6 FM_in_1, J7 Conn_02x08_Odd_Even, J8 Audiojack 1, Q17 BC807, Q2 BC817, Q25 BC858, Q26 BC848, SW2 SW_SP3T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

Commit message: 61354534648
Parts:
- added J1: shmidt trigger 2, Connector_PinHeader_1.27mm:PinHeader_1x02_P1.27mm_Vertical, F.Cu at (212.0, 93.7)
- added J2: shmidt trigger 3, Connector_PinHeader_1.27mm:PinHeader_1x02_P1.27mm_Vertical, F.Cu at (212.0, 99.7)
- added J3: shmidt trigger 4, Connector_PinHeader_1.27mm:PinHeader_1x02_P1.27mm_Vertical, F.Cu at (205.7, 89.0)
- added J4: shmidt trigger 5, Connector_PinHeader_1.27mm:PinHeader_1x02_P1.27mm_Vertical, F.Cu at (199.7, 89.0)
- added J5: shmidt trigger 6, Connector_PinHeader_1.27mm:PinHeader_1x02_P1.27mm_Vertical, F.Cu at (194.0, 89.0)
- moved J14 71.2 mm to (162.3, 118.8)
- moved R59 71.2 mm to (169.8, 115.8)
- moved R64 71.2 mm to (166.0, 115.8)
- moved R82 71.2 mm to (155.0, 115.0)
- moved R85 71.2 mm to (162.2, 115.0)
- moved RV11 71.2 mm to (173.5, 118.8)
- moved J8 70.0 mm to (219.0, 98.5)
- moved U1 66.6 mm to (190.4, 101.0)
- moved U5 66.6 mm to (190.5, 112.2)
- moved D1 65.6 mm to (203.5, 115.6)
- moved R2 65.6 mm to (208.3, 117.6)
- moved R95 65.6 mm to (198.6, 115.4)
- moved C1 65.6 mm to (211.3, 117.6)
- moved C10 65.6 mm to (173.2, 106.6)
- moved C13 65.6 mm to (181.6, 106.1)
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Connections:
- U1 pad 10: (no net) -> Net-(J4-Pin_2)
- U1 pad 11: (no net) -> Net-(J4-Pin_1)
- U1 pad 12: (no net) -> Net-(J5-Pin_2)
- U1 pad 13: (no net) -> Net-(J5-Pin_1)
- U1 pad 3: (no net) -> Net-(J1-Pin_1)
- U1 pad 4: (no net) -> Net-(J1-Pin_2)
- U1 pad 5: (no net) -> Net-(J2-Pin_1)
- U1 pad 6: (no net) -> Net-(J2-Pin_2)
- U1 pad 8: (no net) -> Net-(J3-Pin_2)
- U1 pad 9: (no net) -> Net-(J3-Pin_1)
Routing:
- net SAW_OUT1: track 0.00 -> 57.6 mm
- net Net-(Q25-B): track 0.00 -> 34.9 mm
- net Net-(U2B-+): track 0.00 -> 23.2 mm
- net Net-(U2C--): track 0.00 -> 21.6 mm
- net Net-(D7-K): track 0.00 -> 21.0 mm
- net Net-(D10-A): track 0.00 -> 16.6 mm, vias 0 -> 1
- net TRI_OUT1: track 0.00 -> 13.3 mm
- net CV_IN1: track 0.00 -> 8.51 mm
- net Net-(Q25-E): track 0.00 -> 8.17 mm
- net Net-(R46-Pad1): track 0.00 -> 8.09 mm
- net Net-(R43-Pad1): track 0.00 -> 7.86 mm
- net FM_IN1: track 0.00 -> 7.45 mm
- net Net-(U2A--): track 0.00 -> 7.39 mm
- net Net-(R58-Pad2): track 0.00 -> 6.44 mm
- net PWM_MOD1: track 0.00 -> 6.12 mm
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- added copper zone on In2.Cu, net +12V
- added copper zone on B.Cu, net -12V
- added copper zone on In1.Cu, net GND
Other:
- board outline added: 99 x 38 mm
- board text removed: "TODO: add out connections shmidt trigger"

Commit message: pcb v0.9
Parts:
- J1, J2, J3, J4, J5: footprint Connector_PinHeader_1.27mm:PinHeader_1x02_P1.27mm_Vertical -> Connector_PinHeader_2.00mm:PinHeader_1x02_P2.00mm_Vertical
- moved J5 2.25 mm to (191.8, 89.0)
- moved J4 1.23 mm to (198.5, 89.0)
- moved J3 0.48 mm to (205.2, 89.0)
Routing:
- net Net-(D7-A): track 0.00 -> 35.9 mm, vias 0 -> 1
- net PULSE_OUT1: track 2.09 -> 36.0 mm, vias 0 -> 1
- net OUT1: track 0.00 -> 30.0 mm
- net Net-(D7-K): track 21.0 -> 50.5 mm, vias 0 -> 1
- net Net-(U5A--): track 0.00 -> 22.1 mm
- net Net-(J1-Pin_1): track 0.00 -> 19.6 mm
- net LED_OUT1: track 0.00 -> 19.4 mm
- net +12V: track 5.29 -> 23.4 mm, vias 0 -> 3
- net Net-(J1-Pin_2): track 0.00 -> 16.2 mm
- net Net-(J2-Pin_1): track 0.00 -> 12.4 mm
- net Net-(U5A-+): track 0.00 -> 10.5 mm
- net Net-(J2-Pin_2): track 0.00 -> 10.3 mm
- net GND: track 0.00 -> 8.29 mm
- net Net-(U2D--): track 5.43 -> 13.6 mm, vias 0 -> 1
- net Net-(D1-K): track 0.00 -> 7.38 mm
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- added copper zone on F.Cu, net GND
