File: VCO/VCO_single_osc/VCO_selfetch.kicad_sch (KiCad schematic)
At the start: 41 parts, among them J11 CV_in_1, J14 PWMMOD_in_1, J6 FM_in_1, Q25 BC858, Q26 BC848, U1 40106, U2 TL074

Commit message: 61354534648
Parts:
- added J1: shmidt trigger 2, Connector_PinHeader_1.27mm:PinHeader_1x02_P1.27mm_Vertical, symbol Connector:Conn_01x02_Pin
- added J2: shmidt trigger 3, Connector_PinHeader_1.27mm:PinHeader_1x02_P1.27mm_Vertical, symbol Connector:Conn_01x02_Pin
- added J3: shmidt trigger 4, Connector_PinHeader_1.27mm:PinHeader_1x02_P1.27mm_Vertical, symbol Connector:Conn_01x02_Pin
- added J4: shmidt trigger 5, Connector_PinHeader_1.27mm:PinHeader_1x02_P1.27mm_Vertical, symbol Connector:Conn_01x02_Pin
- added J5: shmidt trigger 6, Connector_PinHeader_1.27mm:PinHeader_1x02_P1.27mm_Vertical, symbol Connector:Conn_01x02_Pin
- added unit 2 of U1
- added unit 4 of U1
- added unit 3 of U1
- added unit 5 of U1
- added unit 6 of U1
Connections:
- new net: J1.1 (Pin_1), U1.3
- new net: J1.2 (Pin_2), U1.4
- new net: J4.1 (Pin_1), U1.11
- new net: J4.2 (Pin_2), U1.10
- new net: J2.1 (Pin_1), U1.5
- new net: J2.2 (Pin_2), U1.6
- new net: J3.2 (Pin_2), U1.8
- new net: J3.1 (Pin_1), U1.9
- new net: J5.1 (Pin_1), U1.13
- new net: J5.2 (Pin_2), U1.12

Commit message: pcb v0.9
Parts:
- J1, J2, J3, J4, J5: footprint Connector_PinHeader_1.27mm:PinHeader_1x02_P1.27mm_Vertical -> Connector_PinHeader_2.00mm:PinHeader_1x02_P2.00mm_Vertical
Changed lines of the file:
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@@
 		)
 		(instances
-			(project ""
+			(project "VCO_selfetch"
 				(path "/6b8d1967-0d10-4b5c-9e39-62e89318329d"
 					(reference "U1")
@@
 			)
 		)
-		(property "Footprint" "Connector_PinHeader_1.27mm:PinHeader_1x02_P1.27mm_Vertical"
+		(property "Footprint" "Connector_PinHeader_2.00mm:PinHeader_1x02_P2.00mm_Vertical"
 			(at 138.43 144.78 0)
 			(effects
@@
 			)
 		)
-		(property "Footprint" "Connector_PinHeader_1.27mm:PinHeader_1x02_P1.27mm_Vertical"
+		(property "Footprint" "Connector_PinHeader_2.00mm:PinHeader_1x02_P2.00mm_Vertical"
 			(at 138.43 111.76 0)
 			(effects
@@
 		)
 		(instances
-			(project ""
+			(project "VCO_selfetch"
 				(path "/6b8d1967-0d10-4b5c-9e39-62e89318329d"
 					(reference "U1")
@@
 		)
 		(instances
-			(project ""
+			(project "VCO_selfetch"
 				(path "/6b8d1967-0d10-4b5c-9e39-62e89318329d"
 					(reference "U1")
@@
 			)
 		)
-		(property "Footprint" "Connector_PinHeader_1.27mm:PinHeader_1x02_P1.27mm_Vertical"
+		(property "Footprint" "Connector_PinHeader_2.00mm:PinHeader_1x02_P2.00mm_Vertical"
 			(at 138.43 129.54 0)
 			(effects
@@
 		)
 		(instances
-			(project ""
+			(project "VCO_selfetch"
 				(path "/6b8d1967-0d10-4b5c-9e39-62e89318329d"
 					(reference "U1")
@@
 			)
 		)
-		(property "Footprint" "Connector_PinHeader_1.27mm:PinHeader_1x02_P1.27mm_Vertical"
+		(property "Footprint" "Connector_PinHeader_2.00mm:PinHeader_1x02_P2.00mm_Vertical"
 			(at 138.43 95.25 0)
 			(effects
@@
 		)
 		(instances
-			(project ""
+			(project "VCO_selfetch"
 				(path "/6b8d1967-0d10-4b5c-9e39-62e89318329d"
 					(reference "J1")
@@
 			)
 		)
-		(property "Footprint" "Connector_PinHeader_1.27mm:PinHeader_1x02_P1.27mm_Vertical"
+		(property "Footprint" "Connector_PinHeader_2.00mm:PinHeader_1x02_P2.00mm_Vertical"
 			(at 138.43 160.02 0)
 			(effects
@@
 		)
 		(instances
-			(project ""
+			(project "VCO_selfetch"
 				(path "/6b8d1967-0d10-4b5c-9e39-62e89318329d"
 					(reference "U1")
